Commit message: Change joint type

File: models/champ_quad_description/urdf/leg/leg.urdf.xacro (robot description, xacro)
@@ -92,5 +92,5 @@
       </collision>
     </link>
-    <joint name="${name}_hip_joint" type="fixed">
+    <joint name="${name}_hip_joint" type="revolute">
       <axis xyz="1 0 0"/>
       <limit effort="25" lower="${-pi}" upper="${pi}" velocity="1.5"/>
@@ -99,5 +99,5 @@
       <origin xyz="${body_to_hip}" rpy="0 0 0"/>
     </joint>
-    <joint name="${name}_upper_leg_joint" type="fixed">
+    <joint name="${name}_upper_leg_joint" type="revolute">
       <axis xyz="0 1 0"/>
       <limit effort="25" lower="${-pi}" upper="${pi}" velocity="1.5"/>
@@ -106,5 +106,5 @@
       <origin xyz="0 0 -${upper_leg_to_lower_leg_z}" rpy="0 0 0"/>
     </joint>
-    <joint name="${name}_lower_leg_joint" type="fixed">
+    <joint name="${name}_lower_leg_joint" type="revolute">
       <axis xyz="0 1 0"/>
       <limit effort="25" lower="${-pi}" upper="${pi}" velocity="1.5"/>
